File: hardware/Schema/unicon_one_pcb.kicad_pcb (KiCad board)
At the start: 2 copper layers, 31 x 45 mm, 75 parts, among them J1 PROG, J2 PWR, J3 SIDE A, J4 SIDE B, U1 LM340MP-5.0, U2 SIP21106-3.3, U3 STM32F051C8Tx, U4 AT24C16, Y1 8MHz, Y2 32768 Hz

Commit message: atskiriame sluoksnyje, kad galima butu atspausdinti, suzymeti visi kontaktai
Other:
- board text added: "1"
- board text added: "10"
- board text added: "11"
- board text added: "12"
- board text added: "12VDC"
- board text added: "13"
- board text added: "14"
- board text added: "15"
- board text added: "16"
- board text added: "17"
- board text added: "18"
- board text added: "19"
- board text added: "2"
- board text added: "20"
- board text added: "3"
- board text added: "3VDC"
- board text added: "4"
- board text added: "5"
- board text added: "5VDC"
- board text added: "6"
- board text added: "7"
- board text added: "8"
- board text added: "9"
- board text added: "BOOT0"
- board text added: "COM"
- board text added: "J1"
- board text added: "J2"
- board text added: "J3"
- board text added: "J4"
- board text added: "NC"
- board text added: "PA0"
- board text added: "PA1"
- board text added: "PA10"
- board text added: "PA11"
- board text added: "PA12"
- board text added: "PA15"
- board text added: "PA2"
- board text added: "PA3"
- board text added: "PA4"
- board text added: "PA5"
- board text added: "PA6"
- board text added: "PA7"
- board text added: "PA8"
- board text added: "PA9"
- board text added: "PB0"
- board text added: "PB1"
- board text added: "PB10"
- board text added: "PB11"
- board text added: "PB12"
- board text added: "PB13"
- board text added: "PB14"
- board text added: "PB15"
- board text added: "PB2"
- board text added: "PB3"
- board text added: "PB4"
- board text added: "PB5"
- board text added: "PB6"
- board text added: "PB7"
- board text added: "PB8"
- board text added: "PB9"
- board text added: "PC13"
- board text added: "PF6"
- board text added: "PF7"
- board text added: "~NRST"
