File: hardware/Schema/unicon.sch (KiCad schematic (older format))
At the start: 96 parts, among them J1 PROG, J2 PWR, J3 SideA, J4 SideB, U1 LM340MP-5.0, U2 SIP21106-3.3, U3 STM32F051C8Tx, U4 AT24C16, U5 ST485B, U6 ULN2003A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

Commit message: pcb paruosimas, schemos pataisymai
Parts:
- removed R22, R23: 47R, resistors:R_0805, symbol R_47R_0805_1%
Connections:
- net ESCL is gone; now on net IO34: R16.1
- net ESDA is gone; now on net IO35: R17.1
- net 3VDC: now also D3.2, D4.2, R16.2, R17.2
- net 5VDC: no longer D3.2, D4.2, R16.2, R17.2
- net ~NRST: now also J1.4 (~NRST), R5.1; no longer R5.2
- net ~NRSTP: now also R5.2; no longer J1.4 (~NRST), R5.1
Other:
- moved on the sheet: C20, D3, D4, R16, R17, R5, U4

Commit message: sugeneruoti gerberiai
Parts:
- J3: value SideA -> SIDE A
- J4: value SideB -> SIDE B
Connections:
- net BOOTA is gone; now on net BOOT0: J4.4 (Pin_4), R1.2
- net BOOT0: no longer C3.1, R1.1, R2.2, U3.44 (BOOT0)
- net PA11: now reaches J4.11 (Pin_11), RN7.8
- net PA11: now also U8.13 (SS/~PL)
- net PA12: now reaches J4.12 (Pin_12), RN7.6
- net PA12: now also U5.2 (~RE), U5.3 (DE)
- net PF6: now reaches J4.9 (Pin_9), RN7.4
- net PF6: now also U8.12 (LATCH)
- net PF7: now reaches J4.10 (Pin_10), RN7.2
- net PA15: now reaches J4.7 (Pin_7), RN6.8
- net PB3: now reaches J4.8 (Pin_8), RN6.6
- net PB4: now reaches J4.5 (Pin_5), RN6.4
- net PB4: now also R18.1
- net PB5: now reaches J4.6 (Pin_6), RN6.2
- net PB5: now also R19.1
- net PB6: now reaches J3.4 (Pin_4), RN5.2
- net PA5: now reaches J3.10 (Pin_10), RN2.6
- net PA5: now also U8.11 (SCK), U9.6 (SCK)
- net PA6: now reaches J3.11 (Pin_11), RN2.4
- net PA6: now also U8.9 (QH), U9.2 (SO)
- net PA7: now reaches J3.12 (Pin_12), RN2.2
- net PA7: now also U9.5 (SI)
- net PA0: now reaches J3.13 (Pin_13), RN3.8
- net PA1: now reaches J3.14 (Pin_14), RN3.6
- net PA2: now reaches J3.15 (Pin_15), RN3.4
- net PA3: now reaches J3.16 (Pin_16), RN3.2
- net PB0: now reaches J3.17 (Pin_17), RN4.8
- net PB0: now also R20.1
- net PB1: now reaches J3.18 (Pin_18), RN4.6
- net PB1: now also R21.1
- net PB2: now reaches J3.19 (Pin_19), RN4.4
- net PB10: now reaches J3.20 (Pin_20), RN4.2
- net PB7: now reaches J3.5 (Pin_5), RN1.8
- net PB8: now reaches J3.6 (Pin_6), RN1.6
- net PB9: now reaches J3.7 (Pin_7), RN1.4
- net PC13: now reaches J3.8 (Pin_8), RN1.2
- net PA4: now reaches J3.9 (Pin_9), RN2.8
- net PA9: now reaches J4.13 (Pin_13), RN8.4
- net PA9: now also U5.4 (DI)
- net PA10: now reaches J4.14 (Pin_14), RN8.2
- net PA10: now also U5.1 (RO)
- net PB15: now reaches J4.15 (Pin_15), RN8.8
- net PA8: now reaches J4.16 (Pin_16), RN8.6
- net PB13: now reaches J4.17 (Pin_17), RN9.4
- net PB13: now also U8.10 (OE)
- net PB14: now reaches J4.18 (Pin_18), RN9.2
- net PB11: now reaches J4.19 (Pin_19), RN9.8
- net PB12: now reaches J4.20 (Pin_20), RN9.6
- net PB12: now also U9.1 (~CS)
- net IO1 renamed A0
- net IO10 renamed B0
- net B0: no longer R20.1
- net IO11 renamed B1
- net B1: no longer R21.1
- net IO12 renamed B2
- net IO13 renamed B8
- net IO14 renamed B9
- net IO15 renamed C13
- net IO16 renamed B10
- net IO17 renamed B11
- net IO18 renamed B14
- net IO19 renamed B15
- net IO2 renamed A1
- net IO20 renamed A8
- net IO21 renamed F7
- net IO22 renamed A15
- net IO23 renamed B3
- net IO24 renamed B4
- net B4: no longer R18.1
- net IO25 renamed B5
- net B5: no longer R19.1
- net IO26 renamed A5
- net A5: no longer U8.11 (SCK), U9.6 (SCK)
- net IO27 renamed A6
- net A6: no longer U8.9 (QH), U9.2 (SO)
- net IO28 renamed A7
- net A7: no longer U9.5 (SI)
- net IO29 renamed A9
- net A9: no longer U5.4 (DI)
- net IO3 renamed A2
- net IO30 renamed A10
- net A10: no longer U5.1 (RO)
- net IO31 renamed A11
- net A11: no longer U8.13 (SS/~PL)
- net IO32 renamed A12
- net A12: no longer U5.2 (~RE), U5.3 (DE)
- net IO33 renamed F6
- net F6: no longer U8.12 (LATCH)
- net IO34 renamed B6
- net IO35 renamed B7
- net IO36 renamed B12
- net B12: no longer U9.1 (~CS)
- net IO37 renamed B13
- net B13: no longer U8.10 (OE)
- net IO4 renamed A3
- net IO9 renamed A4
- new net BT0: C3.1, R1.1, R2.2, U3.44 (BOOT0)
Other:
- moved on the sheet: D2, D5, D6, D7, D8, J2, J3, J4, R32

Commit message: vbat atjungtas nuo 3vdc ir isvestas i J1 jungti
Parts:
- removed C15, C16, C17, C18, C19, C21, C22, C23, C24, C25, C26: 100nF, capacitors:C_0805, symbol C_100n_0805_X7R
- removed R11: 120R, resistors:R_1206, symbol R_120R_1206_1%
- removed R12, R13: 47R, resistors:R_0805, symbol R_47R_0805_1%
- removed R14, R15: 4.7k, resistors:R_0805, symbol R_4.7k_0805_1%
- removed R18, R19, R20, R21: 200k, resistors:R_0805, symbol R_200k_0805_1%
- removed R24, R26, R28, R30: 30k, resistors:R_0805, symbol R_30k_0805_1%
- removed R25, R27, R29, R31: 10k, resistors:R_0805, symbol R_10k_0805_1%
- removed RN10, RN11: 8.2K, resistors:RN1206, symbol RN_8.2K_5%
- removed RN12, RN13: 120R, resistors:RN1206, symbol RN_120R_5%
- removed U5: ST485B, ics:SOIC-8_3.9x4.9mm_Pitch1.27mm, symbol ST485B
- removed U6: ULN2003A, ics:SOIC-16_3.9x9.9mm_Pitch1.27mm, symbol ULN2003A
- removed U7: LM2902M, ics:SOIC-16_3.9x9.9mm_Pitch1.27mm, symbol OP_LM2902M
- removed U8: 74HC589A, ics:SOIC-16_3.9x9.9mm_Pitch1.27mm, symbol 74HC589A
- removed U9: 25AA02E48, ics:SOIC-8_3.9x4.9mm_Pitch1.27mm, symbol 25AA02E48
Connections:
- net 3VDC: no longer U3.1 (VBAT)
- net COM: no longer J2.4 (Pin_4)
- new net VBAT: J2.4 (Pin_4), U3.1 (VBAT)
