File: hardware/Schema/unicon.kicad_pcb (KiCad board)
At the start: 2 copper layers, 95 x 91 mm, 450 parts, among them J1 PROG, J2 PWR, J3 SIDE A, J4 SIDE B, U1 LM340MP-5.0, U2 SIP21106-3.3, U3 STM32F051C8Tx, U4 AT24C16, Y1 8MHz, Y2 32768 Hz

Commit message: alex 20181009
Parts:
- removed the C1 at (167.3, 60.1)
- removed the C1 at (135.3, 60.1)
- removed the C1 at (103.3, 60.1)
- removed the C1 at (167.3, 106.1)
- removed the C1 at (135.3, 106.1)
- removed the C10 at (148.6, 54.3)
- removed the C10 at (180.6, 54.3)
- removed the C10 at (116.6, 54.3)
- removed the C10 at (180.6, 100.3)
- removed the C10 at (148.6, 100.3)
- removed the C11 at (165.0, 81.9)
- removed the C11 at (101.0, 81.9)
- removed the C11 at (133.0, 81.9)
- removed the C11 at (165.0, 127.9)
- removed the C11 at (133.0, 127.9)
- removed the C12 at (165.0, 80.4)
- removed the C12 at (101.0, 80.4)
- removed the C12 at (133.0, 80.4)
- removed the C12 at (165.0, 126.4)
- removed the C12 at (133.0, 126.4)
- removed the C13 at (152.6, 59.8)
- removed the C13 at (184.6, 59.8)
- removed the C13 at (120.6, 59.8)
- removed the C13 at (184.6, 105.8)
- removed the C13 at (152.6, 105.8)
- removed the C14 at (183.3, 56.1)
- removed the C14 at (151.3, 56.1)
- removed the C14 at (119.3, 56.1)
- removed the C14 at (183.3, 102.1)
- removed the C14 at (151.3, 102.1)
- removed the C2 at (185.0, 64.8)
- removed the C2 at (153.0, 64.8)
- removed the C2 at (121.0, 64.8)
- removed the C2 at (185.0, 110.8)
- removed the C2 at (153.0, 110.8)
- removed the C20 at (177.7, 53.6)
- removed the C20 at (145.7, 53.6)
- removed the C20 at (113.7, 53.6)
- removed the C20 at (177.7, 99.6)
- removed the C20 at (145.7, 99.6)
- removed the C3 at (174.9, 72.8)
- removed the C3 at (110.9, 72.8)
- removed the C3 at (142.9, 72.8)
- removed the C3 at (174.9, 118.8)
- removed the C3 at (142.9, 118.8)
- removed the C4 at (175.3, 63.0)
- removed the C4 at (143.3, 63.0)
- removed the C4 at (111.3, 63.0)
- removed the C4 at (175.3, 109.0)
- removed the C4 at (143.3, 109.0)
- removed the C5 at (165.0, 83.5)
- removed the C5 at (101.0, 83.5)
- removed the C5 at (133.0, 83.5)
- removed the C5 at (165.0, 129.5)
- removed the C5 at (133.0, 129.5)
- removed the C6 at (165.0, 85.0)
- removed the C6 at (101.0, 85.0)
- removed the C6 at (133.0, 85.0)
- removed the C6 at (165.0, 131.0)
- removed the C6 at (133.0, 131.0)
- removed the C7 at (164.5, 64.7)
- removed the C7 at (132.5, 64.7)
- removed the C7 at (100.5, 64.7)
- removed the C7 at (164.5, 110.7)
- removed the C7 at (132.5, 110.7)
- removed the C8 at (182.8, 61.3)
- removed the C8 at (150.8, 61.3)
- removed the C8 at (118.8, 61.3)
- removed the C8 at (182.8, 107.3)
- removed the C8 at (150.8, 107.3)
- removed the C9 at (146.7, 54.3)
- removed the C9 at (178.7, 54.3)
- removed the C9 at (114.7, 54.3)
- removed the C9 at (178.7, 100.3)
- removed the C9 at (146.7, 100.3)
- removed the D1 at (171.2, 62.9)
- removed the D1 at (139.2, 62.9)
- removed the D1 at (107.2, 62.9)
- removed the D1 at (171.2, 108.9)
- removed the D1 at (139.2, 108.9)
- removed the D2 at (167.8, 93.5)
- removed the D2 at (103.8, 93.5)
- removed the D2 at (135.8, 93.5)
- removed the D2 at (167.8, 139.5)
- removed the D2 at (135.8, 139.5)
- removed the D3 at (174.7, 53.6)
- removed the D3 at (142.7, 53.6)
- removed the D3 at (110.7, 53.6)
- removed the D3 at (174.7, 99.6)
- removed the D3 at (142.7, 99.6)
- removed the D4 at (171.1, 53.6)
- removed the D4 at (139.1, 53.6)
- removed the D4 at (107.1, 53.6)
- removed the D4 at (171.1, 99.6)
- removed the D4 at (139.1, 99.6)
- removed the D5 at (170.1, 93.5)
- removed the D5 at (106.1, 93.5)
- removed the D5 at (138.1, 93.5)
- removed the D5 at (170.1, 139.5)
- removed the D5 at (138.1, 139.5)
- removed the D6 at (175.9, 93.5)
- removed the D6 at (111.9, 93.5)
- removed the D6 at (143.9, 93.5)
- removed the D6 at (175.9, 139.5)
- removed the D6 at (143.9, 139.5)
- removed the D7 at (178.5, 93.5)
- removed the D7 at (114.5, 93.5)
- removed the D7 at (146.5, 93.5)
- removed the D7 at (178.5, 139.5)
- removed the D7 at (146.5, 139.5)
- removed the D8 at (185.0, 60.6)
- removed the D8 at (153.0, 60.6)
- removed the D8 at (121.0, 60.6)
- removed the D8 at (185.0, 106.6)
- removed the D8 at (153.0, 106.6)
- removed the D9 at (165.6, 55.7)
- removed the D9 at (133.6, 55.7)
- removed the D9 at (101.5, 55.7)
- removed the D9 at (165.6, 101.7)
- removed the D9 at (133.6, 101.7)
- removed the J1 at (168.8, 69.1)
- removed the J1 at (104.8, 69.1)
- removed the J1 at (136.8, 69.1)
- removed the J1 at (168.8, 115.1)
- removed the J1 at (136.8, 115.1)
- removed the J2 at (158.5, 56.9)
- removed the J2 at (126.5, 56.9)
- removed the J2 at (94.5, 56.9)
- removed the J2 at (158.5, 102.9)
- removed the J2 at (126.5, 102.9)
- removed the J3 at (158.5, 69.7)
- removed the J3 at (94.5, 69.7)
- removed the J3 at (126.5, 69.7)
- removed the J3 at (158.5, 115.7)
- removed the J3 at (126.5, 115.7)
- removed the J4 at (183.9, 69.7)
- removed the J4 at (151.9, 69.7)
- removed the J4 at (119.9, 69.7)
- removed the J4 at (183.9, 115.7)
- removed the J4 at (151.9, 115.7)
- removed the R1 at (176.9, 72.8)
- removed the R1 at (112.9, 72.8)
- removed the R1 at (144.9, 72.8)
- removed the R1 at (176.9, 118.8)
- removed the R1 at (144.9, 118.8)
- removed the R10 at (165.2, 53.4)
- removed the R10 at (133.2, 53.4)
- removed the R10 at (101.2, 53.4)
- removed the R10 at (165.2, 99.4)
- removed the R10 at (133.2, 99.4)
- removed the R16 at (180.5, 61.2)
- removed the R16 at (148.5, 61.2)
- removed the R16 at (116.5, 61.2)
- removed the R16 at (180.5, 107.2)
- removed the R16 at (148.5, 107.2)
- removed the R17 at (178.5, 61.2)
- removed the R17 at (146.5, 61.2)
- removed the R17 at (114.5, 61.2)
- removed the R17 at (178.5, 107.2)
- removed the R17 at (146.5, 107.2)
- removed the R2 at (172.9, 72.8)
- removed the R2 at (108.9, 72.8)
- removed the R2 at (140.9, 72.8)
- removed the R2 at (172.9, 118.8)
- removed the R2 at (140.9, 118.8)
- removed the R3 at (168.9, 72.8)
- removed the R3 at (104.9, 72.8)
- removed the R3 at (136.9, 72.8)
- removed the R3 at (168.9, 118.8)
- removed the R3 at (136.9, 118.8)
- removed the R32 at (178.5, 57.3)
- removed the R32 at (146.5, 57.3)
- removed the R32 at (114.5, 57.3)
- removed the R32 at (178.5, 103.3)
- removed the R32 at (146.5, 103.3)
- removed the R4 at (170.9, 72.8)
- removed the R4 at (106.9, 72.8)
- removed the R4 at (138.9, 72.8)
- removed the R4 at (170.9, 118.8)
- removed the R4 at (138.9, 118.8)
- removed the R5 at (180.6, 71.7)
- removed the R5 at (116.6, 71.7)
- removed the R5 at (148.6, 71.7)
- removed the R5 at (180.6, 117.7)
- removed the R5 at (148.6, 117.7)
- removed the R6 at (180.6, 68.6)
- removed the R6 at (116.6, 68.6)
- removed the R6 at (148.6, 68.6)
- removed the R6 at (180.6, 114.6)
- removed the R6 at (148.6, 114.6)
- removed the R7 at (182.8, 64.8)
- removed the R7 at (150.8, 64.8)
- removed the R7 at (118.8, 64.8)
- removed the R7 at (182.8, 110.8)
- removed the R7 at (150.8, 110.8)
- removed the R8 at (146.7, 59.8)
- removed the R8 at (178.7, 59.8)
- removed the R8 at (114.7, 59.8)
- removed the R8 at (178.7, 105.8)
- removed the R8 at (146.7, 105.8)
- removed the R9 at (165.0, 86.5)
- removed the R9 at (101.0, 86.5)
- removed the R9 at (133.0, 86.5)
- removed the R9 at (165.0, 132.5)
- removed the R9 at (133.0, 132.5)
- removed the REF** at (182.1, 69.7)
- removed the REF** at (166.9, 79.0)
- removed the REF** at (163.7, 94.3)
- removed the REF** at (171.8, 76.0)
- removed the REF** at (174.3, 76.1)
- removed the REF** at (174.9, 82.0)
- removed the REF** at (173.5, 86.1)
- removed the REF** at (176.5, 89.3)
- removed the REF** at (177.6, 78.9)
- removed the REF** at (168.5, 78.0)
- removed the REF** at (148.1, 57.2)
- removed the REF** at (166.5, 62.7)
- removed the REF** at (134.5, 62.7)
- removed the REF** at (133.6, 57.2)
- removed the REF** at (139.0, 58.3)
- removed the REF** at (99.7, 94.3)
- removed the REF** at (112.5, 89.3)
- removed the REF** at (110.9, 82.0)
- removed the REF** at (109.5, 86.1)
- removed the REF** at (104.5, 78.0)
- removed the REF** at (102.9, 79.0)
- removed the REF** at (113.6, 78.9)
- removed the REF** at (165.6, 57.2)
- removed the REF** at (107.8, 76.0)
- removed the REF** at (99.8, 73.1)
- removed the REF** at (102.5, 62.7)
- removed the REF** at (101.6, 57.2)
- removed the REF** at (110.3, 76.1)
- removed the REF** at (114.4, 72.9)
- removed the REF** at (107.0, 58.3)
- removed the REF** at (116.1, 57.2)
- removed the REF** at (118.1, 69.7)
- removed the REF** at (150.1, 69.7)
- removed the REF** at (171.0, 58.3)
- removed the REF** at (146.4, 72.9)
- removed the REF** at (136.5, 78.0)
- removed the REF** at (134.9, 79.0)
- removed the REF** at (131.8, 73.1)
- removed the REF** at (145.6, 78.9)
- removed the REF** at (142.9, 82.0)
- removed the REF** at (142.3, 76.1)
- removed the REF** at (139.8, 76.0)
- removed the REF** at (149.7, 83.0)
- removed the REF** at (150.6, 94.3)
- removed the REF** at (180.1, 57.2)
- removed the REF** at (131.7, 94.3)
- removed the REF** at (118.6, 94.3)
- removed the REF** at (117.7, 83.0)
- removed the REF** at (141.5, 86.1)
- removed the REF** at (144.5, 89.3)
- removed the REF** at (180.1, 103.2)
- removed the REF** at (165.6, 103.2)
- removed the REF** at (166.5, 108.7)
- removed the REF** at (171.0, 104.3)
- removed the REF** at (174.3, 122.1)
- removed the REF** at (163.8, 73.1)
- removed the REF** at (171.8, 122.0)
- removed the REF** at (178.4, 118.9)
- removed the REF** at (182.1, 115.7)
- removed the REF** at (182.6, 140.3)
- removed the REF** at (181.7, 129.0)
- removed the REF** at (173.5, 132.1)
- removed the REF** at (177.6, 124.9)
- removed the REF** at (176.5, 135.3)
- removed the REF** at (168.5, 124.0)
- removed the REF** at (166.9, 125.0)
- removed the REF** at (178.4, 72.9)
- removed the REF** at (174.9, 128.0)
- removed the REF** at (163.8, 119.1)
- removed the REF** at (163.7, 140.3)
- removed the REF** at (148.1, 103.2)
- removed the REF** at (133.6, 103.2)
- removed the REF** at (134.5, 108.7)
- removed the REF** at (139.0, 104.3)
- removed the REF** at (142.3, 122.1)
- removed the REF** at (139.8, 122.0)
- removed the REF** at (146.4, 118.9)
- removed the REF** at (182.6, 94.3)
- removed the REF** at (150.1, 115.7)
- removed the REF** at (150.6, 140.3)
- removed the REF** at (149.7, 129.0)
- removed the REF** at (141.5, 132.1)
- removed the REF** at (145.6, 124.9)
- removed the REF** at (144.5, 135.3)
- removed the REF** at (136.5, 124.0)
- removed the REF** at (134.9, 125.0)
- removed the REF** at (142.9, 128.0)
- removed the REF** at (131.8, 119.1)
- removed the REF** at (181.7, 83.0)
- removed the REF** at (131.7, 140.3)
- removed the RN1 at (163.8, 75.6)
- removed the RN1 at (99.8, 75.6)
- removed the RN1 at (131.8, 75.6)
- removed the RN1 at (163.8, 121.6)
- removed the RN1 at (131.8, 121.6)
- removed the RN14 at (173.0, 93.2)
- removed the RN14 at (109.0, 93.2)
- removed the RN14 at (141.0, 93.2)
- removed the RN14 at (173.0, 139.2)
- removed the RN14 at (141.0, 139.2)
- removed the RN2 at (163.8, 80.7)
- removed the RN2 at (99.8, 80.7)
- removed the RN2 at (131.8, 80.7)
- removed the RN2 at (163.8, 126.7)
- removed the RN2 at (131.8, 126.7)
- removed the RN3 at (163.8, 85.8)
- removed the RN3 at (99.8, 85.8)
- removed the RN3 at (131.8, 85.8)
- removed the RN3 at (163.8, 131.8)
- removed the RN3 at (131.8, 131.8)
- removed the RN4 at (163.8, 90.7)
- removed the RN4 at (99.8, 90.7)
- removed the RN4 at (131.8, 90.7)
- removed the RN4 at (163.8, 136.7)
- removed the RN4 at (131.8, 136.7)
- removed the RN5 at (163.8, 70.6)
- removed the RN5 at (99.8, 70.6)
- removed the RN5 at (131.8, 70.6)
- removed the RN5 at (163.8, 116.6)
- removed the RN5 at (131.8, 116.6)
- removed the RN6 at (181.1, 75.5)
- removed the RN6 at (117.1, 75.5)
- removed the RN6 at (149.1, 75.5)
- removed the RN6 at (181.1, 121.5)
- removed the RN6 at (149.1, 121.5)
- removed the RN7 at (181.1, 80.6)
- removed the RN7 at (117.1, 80.6)
- removed the RN7 at (149.1, 80.6)
- removed the RN7 at (181.1, 126.6)
- removed the RN7 at (149.1, 126.6)
- removed the RN8 at (181.1, 85.7)
- removed the RN8 at (149.1, 85.7)
- removed the RN8 at (117.1, 85.7)
- removed the RN8 at (181.1, 131.7)
- removed the RN8 at (149.1, 131.7)
- removed the RN9 at (181.1, 90.8)
- removed the RN9 at (117.1, 90.8)
- removed the RN9 at (149.1, 90.8)
- removed the RN9 at (181.1, 136.8)
- removed the RN9 at (149.1, 136.8)
- removed the U1 at (141.7, 56.5)
- removed the U1 at (173.7, 56.5)
- removed the U1 at (109.7, 56.5)
- removed the U1 at (173.7, 102.5)
- removed the U1 at (141.7, 102.5)
- removed the U2 at (149.7, 59.8)
- removed the U2 at (181.7, 59.8)
- removed the U2 at (117.7, 59.8)
- removed the U2 at (181.7, 105.8)
- removed the U2 at (149.7, 105.8)
- removed the U3 at (172.8, 84.8)
- removed the U3 at (108.8, 84.8)
- removed the U3 at (140.8, 84.8)
- removed the U3 at (172.8, 130.8)
- removed the U3 at (140.8, 130.8)
- removed the U4 at (173.7, 58.3)
- removed the U4 at (141.7, 58.3)
- removed the U4 at (109.7, 58.3)
- removed the U4 at (173.7, 104.3)
- removed the U4 at (141.7, 104.3)
- removed the Y1 at (170.0, 86.2)
- removed the Y1 at (106.0, 86.2)
- removed the Y1 at (138.0, 86.2)
- removed the Y1 at (170.0, 132.2)
- removed the Y1 at (138.0, 132.2)
- removed the Y2 at (176.2, 81.0)
- removed the Y2 at (112.2, 81.0)
- removed the Y2 at (144.2, 81.0)
- removed the Y2 at (176.2, 127.0)
- removed the Y2 at (144.2, 127.0)
Routing:
- net /3VDC: track 827.5 -> 137.9 mm, vias 18 -> 3
- net /5VDC: track 376.7 -> 62.8 mm
- net /~NRST: track 279.5 -> 46.6 mm, vias 18 -> 3
- net /B6: track 277.8 -> 46.3 mm, vias 24 -> 4
- net /B7: track 261.1 -> 43.5 mm
- net /VDDA: track 212.2 -> 35.4 mm, vias 12 -> 2
- net /A6: track 155.6 -> 25.9 mm, vias 12 -> 2
- net /A5: track 148.6 -> 24.8 mm, vias 12 -> 2
- net /A4: track 143.2 -> 23.9 mm, vias 12 -> 2
- net /SWDIO: track 125.3 -> 20.9 mm, vias 12 -> 2
- net /B10: track 119.8 -> 20.0 mm, vias 12 -> 2
- net /B2: track 119.1 -> 19.9 mm, vias 12 -> 2
- net /OSC32_I: track 113.5 -> 18.9 mm, vias 6 -> 1
- net /B1: track 111.2 -> 18.5 mm, vias 12 -> 2
- net Net-(C1-Pad1): track 105.8 -> 17.6 mm, vias 6 -> 1
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Other:
- board size 95 x 91 mm -> 31 x 45 mm
- board text added: "1"
- board text added: "10"
- board text added: "11"
- board text added: "12"
- board text added: "12VDC"
- board text added: "13"
- board text added: "14"
- board text added: "15"
- board text added: "16"
- board text added: "17"
- board text added: "18"
- board text added: "19"
- board text added: "2"
- board text added: "20"
- board text added: "3"
- board text added: "3VDC"
- board text added: "4"
- board text added: "5"
- board text added: "5VDC"
- board text added: "6"
- board text added: "7"
- board text added: "8"
- board text added: "9"
- board text added: "BOOT0"
- board text added: "COM"
- board text added: "J1"
- board text added: "J2"
- board text added: "J3"
- board text added: "J4"
- board text added: "NC"
- board text added: "PA0"
- board text added: "PA1"
- board text added: "PA10"
- board text added: "PA11"
- board text added: "PA12"
- board text added: "PA15"
- board text added: "PA2"
- board text added: "PA3"
- board text added: "PA4"
- board text added: "PA5"
- board text added: "PA6"
- board text added: "PA7"
- board text added: "PA8"
- board text added: "PA9"
- board text added: "PB0"
- board text added: "PB1"
- board text added: "PB10"
- board text added: "PB11"
- board text added: "PB12"
- board text added: "PB13"
- board text added: "PB14"
- board text added: "PB15"
- board text added: "PB2"
- board text added: "PB3"
- board text added: "PB4"
- board text added: "PB5"
- board text added: "PB6"
- board text added: "PB7"
- board text added: "PB8"
- board text added: "PB9"
- board text added: "PC13"
- board text added: "PF6"
- board text added: "PF7"
- board text added: "~NRST"
