File: hardware/Schema/unicon.kicad_pcb (KiCad board)
At the start: 2 copper layers, 31 x 45 mm, 75 parts, among them J1 PROG, J2 PWR, J3 SIDE A, J4 SIDE B, U1 LM340MP-5.0, U2 SIP21106-3.3, U3 STM32F051C8Tx, U4 AT24C16, Y1 8MHz, Y2 32768 Hz

Commit message: 20181012
Parts:
- D2: value LED1 -> LED2
- D5: value LED2 -> LED5
- D6: value LED1 -> LED6
- D7: value LED2 -> LED7
- D8: value 3V -> POWER
Connections:
- net Net-(J3-Pad1) renamed /J3.1
- net Net-(J3-Pad2) renamed /J3.2
- net Net-(J3-Pad3) renamed /J3.3
