File: hardware/unicon.kicad_pcb (KiCad board)
At the start: 2 copper layers, 31 x 45 mm, 75 parts, among them J1 PROG, J2 PWR, J3 SIDE A, J4 SIDE B, U1 LM340MP-5.0, U2 SIP21106-3.3, U3 STM32F051C8Tx, U4 AT24C16, Y1 8MHz, Y2 32768 Hz

Commit message: isvestas i isore VBAT
Parts:
- moved REF** 0.78 mm to (105.3, 124.1)
- moved REF** 0.16 mm to (102.9, 125.2)
Connections:
- J2 pad 4: /COM -> /VBAT
- RN5 pad 3: (no net) -> Net-(RN5-Pad3)
- RN5 pad 5: (no net) -> Net-(RN5-Pad5)
- RN5 pad 7: (no net) -> Net-(RN5-Pad7)
- U3 pad 1: /3VDC -> /VBAT
Routing:
- net /VBAT: track 0.00 -> 30.1 mm, vias 0 -> 1
- net /3VDC: track 137.9 -> 136.3 mm
- net /OSC32_I: track 18.9 -> 19.6 mm
