File: hardware/unicon.sch (KiCad schematic (older format))
At the start: 57 parts, among them J1 PROG, J2 PWR, J3 SIDE A, J4 SIDE B, U1 LM340MP-5.0, U2 SIP21106-3.3, U3 STM32F051C8Tx, U4 AT24C16, Y1 8MHz, Y2 32768 Hz

Commit message: isvestas i isore VBAT
Connections:
- net labels added: VBAT
- wire segments 334 -> 333
Changed lines of the file:
@@
 LIBS:various
 LIBS:resistors
-LIBS:LED
 LIBS:power
 LIBS:device
@@
 VDDA
 Text Label 5200 3700 0    50   ~ 0
-3VDC
+VBAT
 Text Label 6500 2750 3    50   ~ 0
 BT0
@@
 	1775 5150 2525 5150
 Wire Wire Line
-	2525 4850 2525 4950
-Wire Wire Line
-	2525 4850 2400 4850
+	2800 4850 2400 4850
 Wire Wire Line
 	2400 4950 2525 4950
-Connection ~ 2525 4950
 Connection ~ 2525 5150
 Wire Wire Line
@@
 Text Label 2600 5400 2    50   ~ 0
 J3.2
+Text Label 2800 4850 2    50   ~ 0
+VBAT
 $EndSCHEMATC
